File: SE/Semáforo/Semáforo.brd (EAGLE design)
At the start: 134.5 x 59.7 mm, 7 parts, among them U2 ARDUINO-UNO-R3-SHIELD

Commit message: SI - Sistema de semáforo atualizado
Agora o sistema de semáforo tem os leds para as pessoas, com as cores vermelho e azul
Parts:
- added D1: GREEN, Tinkercad:LEDRD254W60D565H860B_G
- added D2: RED, Tinkercad:LEDRD254W60D565H860B
- added R1, R2: 1k, Tinkercad:RESAD1016W63L850D250B
Connections:
- new net D1_C: D1.2, R1.2
- new net D2_C: D2.2, R2.2
- new net U2_D5: D1.1, U2.D5
- new net U2_D6: D2.1, U2.D6
- net U2_GND: now also R1.1, R2.1
Other:
- board size 134.5 x 59.7 mm -> 172.6 x 59.7 mm
